Commit message: The simulation file should be able to read from a list and display it now

File: exo-urdf/01-exo_arm.urdf (robot description, URDF)
Before this commit: robot visual, 2 links, 1 joints
Joints:
- joint base_to_forearm: limit lower=0.0 upper=2 effort=1000.0 velocity=0.5 -> lower=0.0 upper=2 effort=1000.0 velocity=2.0
